Commit message: Back up of current working model.

File: description/lidar.xacro (robot description, xacro)
@@ -3,56 +3,59 @@
     <joint name="laser_joint" type="fixed">
         <parent link="chassis"/>
-        <child link="lidar_link"/>
+        <child link="laser_frame"/>
         <origin xyz="0.27 0 0.07" rpy="0 0 0"/>
     </joint>
-    <link name="lidar_link">
-            <visual>
-                <origin xyz="0.0 0.0 0.0" rpy="0.0 0.0 0.0"/>
-                <geometry>
-                    <cylinder radius="0.05" length="0.04"/>
-                </geometry>
-                <material name="red"/>
-            </visual>
-            <collision>
-                <origin xyz="0.0 0.0 0.0" rpy="0.0 0.0 0.0"/>
-                <geometry>
-                    <cylinder radius="0.05" length="0.04"/>
-                </geometry>
-            </collision>
-            <xacro:inertial_cylinder mass="1" radius="0.05" length="0.04">
-                <origin xyz="0.0 0.0 0.0" rpy="0.0 0.0 0.0"/>
-            </xacro:inertial_cylinder>
-        </link>
-        <gazebo reference="lidar_link">
-            <material>Gazebo/FlatBlack</material>
-            <sensor type="ray" name="lidar_sensor">
-                <pose>0 0 0 0 0 0</pose>
-                <visualize>true</visualize>
-                <update_rate>30</update_rate>
-                <ray>
-                    <scan>
-                        <horizontal>
-                            <samples>360</samples>
-                            <resolution>1</resolution>
-                            <min_angle>-3.14</min_angle>
-                            <max_angle>3.14</max_angle>
-                        </horizontal>
-                    </scan>
-                    <range>
-                        <min>0.3</min>
-                        <max>12</max>
-                        <resolution>0.01</resolution>
-                    </range>
-                    <!-- <noise>
-                        <type>gaussian</type>
-                        <mean>0.0</mean>
-                        <stddev>0.01</stddev>
-                    </noise> -->
-                </ray>
-                <plugin name="gazebo_ros_lidar_controller" filename="libgazebo_ros_laser.so">
-                    <topicName>scan</topicName>
-                    <frameName>lidar_link</frameName>
-                </plugin>
-            </sensor>
-        </gazebo>
+    <link name="laser_frame">
+        <visual>
+            <origin xyz="0.0 0.0 0.0" rpy="0.0 0.0 0.0"/>
+            <geometry>
+                <cylinder radius="0.05" length="0.04"/>
+            </geometry>
+            <material name="red"/>
+        </visual>
+        <collision>
+            <origin xyz="0.0 0.0 0.0" rpy="0.0 0.0 0.0"/>
+            <geometry>
+                <cylinder radius="0.05" length="0.04"/>
+            </geometry>
+        </collision>
+        <xacro:inertial_cylinder mass="1" radius="0.05" length="0.04">
+            <origin xyz="0.0 0.0 0.0" rpy="0.0 0.0 0.0"/>
+        </xacro:inertial_cylinder>
+    </link>
+    <gazebo reference="laser_frame">
+        <material>Gazebo/FlatBlack</material>
+        <sensor type="ray" name="laser">
+            <pose>0 0 0 0 0 0</pose>
+            <visualize>true</visualize>
+            <update_rate>30</update_rate>
+            <ray>
+                <scan>
+                    <horizontal>
+                        <samples>360</samples>
+                        <resolution>1</resolution>
+                        <min_angle>-3.14</min_angle>
+                        <max_angle>3.14</max_angle>
+                    </horizontal>
+                </scan>
+                <range>
+                    <min>0.3</min>
+                    <max>12</max>
+                    <resolution>0.01</resolution>
+                </range>
+                <!-- <noise>
+                    <type>gaussian</type>
+                    <mean>0.0</mean>
+                    <stddev>0.01</stddev>
+                </noise> -->
+            </ray>
+            <plugin name="laser_controller" filename="libgazebo_ros_ray_sensor.so">
+                <ros>
+                    <!-- <argument>~/out:=scan</argument> -->
+                    <argument>--ros-args -r ~/out:=scan</argument>
+                </ros>
+                <output_type>sensor_msgs/LaserScan</output_type>
+            </plugin>
+        </sensor>
+    </gazebo>
 </robot>

File: description/robot.urdf.xacro (robot description, xacro)
@@ -4,3 +4,4 @@
     <!-- <xacro:include filename="$(find ford_bot)/description/test_robot.xacro"/> -->
     <xacro:include filename="lidar.xacro"/>
+    <xacro:include filename="gazebo_control.xacro"/>
 </robot>

File: description/robot_core.xacro (robot description, xacro)
@@ -2,5 +2,4 @@
 <robot xmlns:xacro="http://www.ros.org/wiki/xacro">
     <xacro:include filename="inertial_macros.xacro"/>
-    <xacro:include filename="gazebo_control.xacro"/>
     <!-- <xacro:include filename="lidar.xacro"/> -->
     <material name="white">
