Commit message: Slam_toolbox added and works for the most part.

File: description/gazebo_control.xacro (robot description, xacro)
@@ -4,25 +4,25 @@
         <mu1>0.2</mu1>
         <mu2>0.2</mu2>
-        <material>Gazebo/Green</material>
+        <material>Gazebo/Silver</material>
     </gazebo>
     <gazebo reference="front_right_wheel">
         <mu1>0.2</mu1>
         <mu2>0.2</mu2>
-        <material>Gazebo/White</material>
+        <material>Gazebo/Orange</material>
     </gazebo>
     <gazebo reference="front_left_wheel">
         <mu1>0.2</mu1>
         <mu2>0.2</mu2>
-        <material>Gazebo/White</material>
+        <material>Gazebo/Orange</material>
     </gazebo>
     <gazebo reference="rear_right_wheel">
         <mu1>0.2</mu1>
         <mu2>0.2</mu2>
-        <material>Gazebo/White</material>
+        <material>Gazebo/Orange</material>
     </gazebo>
     <gazebo reference="rear_left_wheel">
         <mu1>0.2</mu1>
         <mu2>0.2</mu2>
-        <material>Gazebo/White</material>
+        <material>Gazebo/Orange</material>
     </gazebo>
 <!-- Controller for the 4-wheeled robot -->

File: description/lidar.xacro (robot description, xacro)
@@ -4,5 +4,5 @@
         <parent link="chassis"/>
         <child link="laser_frame"/>
-        <origin xyz="0.27 0 0.07" rpy="0 0 0"/>
+        <origin xyz="0.22 0 0.222" rpy="0 0 0"/>
     </joint>
     <link name="laser_frame">
@@ -44,16 +44,12 @@
                     <resolution>0.01</resolution>
                 </range>
-                <!-- <noise>
-                    <type>gaussian</type>
-                    <mean>0.0</mean>
-                    <stddev>0.01</stddev>
-                </noise> -->
             </ray>
             <plugin name="laser_controller" filename="libgazebo_ros_ray_sensor.so">
                 <ros>
-                    <!-- <argument>~/out:=scan</argument> -->
-                    <argument>--ros-args -r ~/out:=scan</argument>
+                    <argument>~/out:=scan</argument>
+                    <!-- <argument>ros-args -r ~/out:=scan</argument> -->
                 </ros>
                 <output_type>sensor_msgs/LaserScan</output_type>
+                <frame_name>laser_frame</frame_name>
             </plugin>
         </sensor>

File: description/robot.urdf.xacro (robot description, xacro)
@@ -1,6 +1,6 @@
 <?xml version="1.0"?>
 <robot xmlns:xacro="http://www.ros.org/wiki/xacro" name="ford_robot">
-    <xacro:include filename="robot_core.xacro"/>
-    <!-- <xacro:include filename="$(find ford_bot)/description/test_robot.xacro"/> -->
+    <!-- <xacro:include filename="robot_core.xacro"/> -->
+    <xacro:include filename="mecabot.xacro"/>
     <xacro:include filename="lidar.xacro"/>
     <xacro:include filename="gazebo_control.xacro"/>
